File: ps2-pms.kicad_sch (KiCad schematic)
At the start: 87 parts, among them U1 ADP151, U2 SC174, U3 TPS61253

Commit message: docs(added-BOM): Added Bill of materials
Parts:
- C16: value (none) -> 47uF
- S?: value (none) -> button
- gave numbers to parts that had none: 1
- renumbered C1 to C101
Changed lines of the file:
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@@
       (effects (font (size 1.27 1.27)) (justify right))
     )
-    (property "Value" "" (id 1) (at 160.02 39.37 90)
+    (property "Value" "button" (id 1) (at 160.02 39.37 90)
       (effects (font (size 1.27 1.27)) (justify right))
     )
@@
   (symbol (lib_id "ps2-pms:bq2407x") (at 147.32 113.03 0) (unit 1)
     (in_bom yes) (on_board yes)
-    (property "Reference" "U?" (id 0) (at 147.32 113.03 0))
+    (property "Reference" "U4" (id 0) (at 147.32 113.03 0))
     (property "Value" "bq2407x" (id 1) (at 147.32 109.22 0))
     (property "Footprint" "" (id 2) (at 147.32 113.03 0)
@@
   (symbol (lib_id "Device:C_Polarized_Small_US") (at 262.89 22.86 0) (unit 1)
     (in_bom yes) (on_board yes)
-    (property "Reference" "C1" (id 0) (at 265.43 21.59 0)
+    (property "Reference" "C101" (id 0) (at 265.43 21.59 0)
       (effects (font (size 1.27 1.27)) (justify left))
     )
@@
       (effects (font (size 1.27 1.27)) (justify left))
     )
-    (property "Value" "" (id 1) (at 179.07 43.18 0)
+    (property "Value" "47uF" (id 1) (at 179.07 43.18 0)
       (effects (font (size 1.27 1.27)) (justify left))
     )
@@
       (reference "BT?") (unit 1) (value "Battery_Cell") (footprint "")
     )
-    (path "/9d72ec0b-ea88-439d-b756-f0d0a946897f"
-      (reference "C1") (unit 1) (value "1µF") (footprint "")
-    )
     (path "/c9ca6bc0-254d-4703-8256-9c8ce6c5a9a7"
       (reference "C1") (unit 1) (value "1µF") (footprint "")
@@
       (reference "C16") (unit 1) (value "47uF") (footprint "")
     )
+    (path "/9d72ec0b-ea88-439d-b756-f0d0a946897f"
+      (reference "C101") (unit 1) (value "1µF") (footprint "")
+    )
     (path "/17920d38-4202-4d9b-a3fe-7fc83f322ad5"
       (reference "C?") (unit 1) (value "22uF/6.3v") (footprint "")
@@
       (reference "U3") (unit 1) (value "TPS61253") (footprint "")
     )
+    (path "/96aaca5e-0f64-4799-8bc0-ad1b6aca8450"
+      (reference "U4") (unit 1) (value "bq2407x") (footprint "")
+    )
     (path "/0108fbbd-bb2f-4247-9e7c-8ed949a2604f"
       (reference "U?") (unit 1) (value "BC847C") (footprint "")
@@
       (reference "U?") (unit 1) (value "TL431") (footprint "")
     )
-    (path "/96aaca5e-0f64-4799-8bc0-ad1b6aca8450"
-      (reference "U?") (unit 1) (value "bq2407x") (footprint "")
-    )
     (path "/b04075d2-3602-43e6-92be-9dd21513a200"

Commit message: build(pms-board): 2.0 build with cleaner contacts, universal ground, and BOM
Parts:
- gave numbers to parts that had none: 2
Changed lines of the file:
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@@
   )
   (symbol (lib_id "Transistor_FET:AO3401A") (at 148.59 67.31 180) (unit 1)
-    (in_bom yes) (on_board yes) (fields_autoplaced)
-    (property "Reference" "Q?" (id 0) (at 142.24 66.0399 0)
+    (in_bom yes) (on_board yes)
+    (property "Reference" "CSD22202W15" (id 0) (at 139.7 66.04 0)
       (effects (font (size 1.27 1.27)) (justify left))
     )
@@
   (symbol (lib_id "Device:Q_NPN_BCE") (at 172.72 31.75 90) (unit 1)
     (in_bom yes) (on_board yes)
-    (property "Reference" "Q?" (id 0) (at 171.45 26.67 0)
+    (property "Reference" "BC846A" (id 0) (at 171.45 26.67 0)
       (effects (font (size 1.27 1.27)) (justify left))
     )
@@
   (symbol (lib_id "Device:Q_NPN_BCE") (at 162.56 62.23 180) (unit 1)
     (in_bom yes) (on_board yes)
-    (property "Reference" "Q?" (id 0) (at 173.99 63.5 0)
+    (property "Reference" "BC846A" (id 0) (at 173.99 63.5 0)
       (effects (font (size 1.27 1.27)) (justify left))
     )
@@
       (reference "#PWR?") (unit 1) (value "GND") (footprint "")
     )
+    (path "/5405a41e-5337-4297-8bac-d2336ab934c1"
+      (reference "BC846A") (unit 1) (value "Q_NPN_BCE") (footprint "")
+    )
+    (path "/fdd46e6f-eeb8-49c8-b304-5c975f4f1f28"
+      (reference "BC846A") (unit 1) (value "Q_NPN_BCE") (footprint "")
+    )
     (path "/5ee98f39-103a-49e6-8d09-c67de3099482"
       (reference "BT?") (unit 1) (value "Battery_Cell") (footprint "")
@@
       (reference "C?") (unit 1) (value "10uF/6.3V") (footprint "")
     )
+    (path "/297294a8-d3af-4a2a-b2ff-ea991d460add"
+      (reference "CSD22202W15") (unit 1) (value "P-channel mosfet") (footprint "Package_TO_SOT_SMD:SOT-23")
+    )
     (path "/8863e1d8-08ba-4f33-9d6e-204128050245"
       (reference "D?") (unit 1) (value "LED_ARBG") (footprint "")
@@
       (reference "L?") (unit 1) (value "2.0uH") (footprint "")
     )
-    (path "/297294a8-d3af-4a2a-b2ff-ea991d460add"
-      (reference "Q?") (unit 1) (value "P-channel mosfet") (footprint "Package_TO_SOT_SMD:SOT-23")
-    )
-    (path "/5405a41e-5337-4297-8bac-d2336ab934c1"
-      (reference "Q?") (unit 1) (value "Q_NPN_BCE") (footprint "")
-    )
-    (path "/fdd46e6f-eeb8-49c8-b304-5c975f4f1f28"
-      (reference "Q?") (unit 1) (value "Q_NPN_BCE") (footprint "")
-    )
     (path "/6b9147be-ef3f-40e6-b07f-fb9b1328bed0"

Commit message: build(final-push): final push
Parts:
- gave numbers to parts that had none: 1
Changed lines of the file:
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@@
   (symbol (lib_id "ps2-pms:TL431") (at 231.14 132.08 270) (unit 1)
     (in_bom yes) (on_board yes)
-    (property "Reference" "U?" (id 0) (at 232.4101 138.43 90)
+    (property "Reference" "U5" (id 0) (at 229.87 133.35 90)
       (effects (font (size 1.27 1.27)) (justify left))
     )
@@
       (reference "U4") (unit 1) (value "bq2407x") (footprint "")
     )
+    (path "/9589205f-693b-42a2-bb81-726f69a2e554"
+      (reference "U5") (unit 1) (value "TL431") (footprint "")
+    )
     (path "/0108fbbd-bb2f-4247-9e7c-8ed949a2604f"
       (reference "U?") (unit 1) (value "BC847C") (footprint "")
@@
       (reference "U?") (unit 1) (value "SC174") (footprint "ps2-pms:SC174")
     )
-    (path "/9589205f-693b-42a2-bb81-726f69a2e554"
-      (reference "U?") (unit 1) (value "TL431") (footprint "")
-    )
     (path "/b04075d2-3602-43e6-92be-9dd21513a200"
